Commit message: US_14441: Snower stl file

File: Software/ros2_ws/src/robot/urdf/ouster_lidar.xacro (robot description, xacro)
@@ -4,8 +4,8 @@
     <parent link="base_link" />
     <child link="os_sensor" />
-    <origin xyz="0.3 0 0.753" />
+    <origin xyz="0.275 0.01 0.73" />
   </joint>
   <link name="os_sensor">
-    <visual>
+    <!-- <visual>
       <origin xyz="0 0 0" />
       <geometry>
@@ -20,5 +20,5 @@
       </geometry>
       <material name="orange" />
-    </visual>
+    </visual> -->
     <collision>
       <origin xyz="0 0 0" />

File: Software/ros2_ws/src/robot/urdf/snower_core.xacro (robot description, xacro)
@@ -36,5 +36,5 @@
     </joint>
     <link name="chassis_link">
-        <visual>
+        <!-- <visual>
             <origin xyz="0 0 0" />
             <geometry>
@@ -42,11 +42,11 @@
             </geometry>
             <material name="white" />
-        </visual>
+        </visual> -->
         <visual>
-            <origin xyz="0.3 0 0.31" />
+            <origin xyz="0 0 -0.245" rpy="0 0 0"/>
             <geometry>
-                <cylinder radius="0.05" length="0.3" />
+                <mesh filename="https://raw.githubusercontent.com/Lapland-Robotics/AI.R-Autonomous_Robot/documentation/3D%20Modeling/Snower_whole_3d.stl"/>
             </geometry>
-            <material name="white" />
+            <material name="orange" />
         </visual>
         <collision>
@@ -73,10 +73,10 @@
     </joint>
     <link name="left_back_wheel_link">
-        <visual>
+        <!-- <visual>
             <geometry>
                 <cylinder radius="0.15" length="0.30" />
             </geometry>
             <material name="black" />
-        </visual>
+        </visual> -->
         <collision>
             <geometry>
@@ -94,10 +94,10 @@
     </joint>
     <link name="right_back_wheel_link">
-        <visual>
+        <!-- <visual>
             <geometry>
                 <cylinder radius="0.15" length="0.30" />
             </geometry>
             <material name="black" />
-        </visual>
+        </visual> -->
         <collision>
             <geometry>
@@ -115,10 +115,10 @@
     </joint>
     <link name="left_front_wheel_link">
-        <visual>
+        <!-- <visual>
             <geometry>
                 <cylinder radius="0.15" length="0.30" />
             </geometry>
             <material name="black" />
-        </visual>
+        </visual> -->
         <collision>
             <geometry>
@@ -136,10 +136,10 @@
     </joint>
     <link name="right_front_wheel_link">
-        <visual>
+        <!-- <visual>
             <geometry>
                 <cylinder radius="0.15" length="0.30" />
             </geometry>
             <material name="black" />
-        </visual>
+        </visual> -->
         <collision>
             <geometry>

File: Software/ros2_ws/src/robot/urdf/zed2_camara.xacro (robot description, xacro)
@@ -4,8 +4,8 @@
         <parent link="base_link" />
         <child link="zed_camera_link" />
-        <origin xyz="0.445 0 0.4165" />
+        <origin xyz="0.442 0 0.41" />
     </joint>
     <link name="zed_camera_link">
-        <visual>
+        <!-- <visual>
             <origin xyz="0 0 0" />
             <geometry>
@@ -13,5 +13,5 @@
             </geometry>
             <material name="orange" />
-        </visual>
+        </visual> -->
         <collision>
             <origin xyz="0 0 0" />

File: Software/ros2_ws/src/robot/urdf/zedf9p_gnss.xacro (robot description, xacro)
@@ -4,8 +4,8 @@
         <parent link="base_link" />
         <child link="gnss_link" />
-        <origin xyz="-0.41 0.2 0.413" />
+        <origin xyz="-0.41 0.16 0.413" />
     </joint>
     <link name="gnss_link">
-        <visual>
+        <!-- <visual>
             <origin xyz="0 0 0" />
             <geometry>
@@ -13,5 +13,5 @@
             </geometry>
             <material name="orange" />
-        </visual>
+        </visual> -->
         <collision>
             <origin xyz="0 0 0" />
