Commit message: US_14441: Snower correct wheel tf origin xyz

File: Software/ros2_ws/src/robot/urdf/snower_core.xacro (robot description, xacro)
@@ -69,5 +69,5 @@
         <parent link="base_link" />
         <child link="left_back_wheel_link" />
-        <origin xyz="-0.26 0.41 0.15" rpy="-${pi/2} 0 0" />
+        <origin xyz="-0.136 0.313 0.142" rpy="0 0 0" />
         <axis xyz="0 0 1" />
     </joint>
@@ -90,5 +90,5 @@
         <parent link="base_link" />
         <child link="right_back_wheel_link" />
-        <origin xyz="-0.26 -0.41 0.15" rpy="${pi/2} 0 0" />
+        <origin xyz="-0.136 -0.313 0.142" rpy="0 0 0" />
         <axis xyz="0 0 -1" />
     </joint>
@@ -111,5 +111,5 @@
         <parent link="base_link" />
         <child link="left_front_wheel_link" />
-        <origin xyz="0.26 0.41 0.15" rpy="-${pi/2} 0 0" />
+        <origin xyz="0.136 0.307 0.142" rpy="0 0 0" />
         <axis xyz="0 0 1" />
     </joint>
@@ -132,5 +132,5 @@
         <parent link="base_link" />
         <child link="right_front_wheel_link" />
-        <origin xyz="0.26 -0.41 0.15" rpy="${pi/2} 0 0" />
+        <origin xyz="0.136 -0.307 0.142" rpy="0 0 0" />
         <axis xyz="0 0 -1" />
     </joint>

Commit message: US_14441: basile final modifications for the robosense lidar

File: Software/ros2_ws/src/robot/urdf/snower_core.xacro (robot description, xacro)
@@ -14,5 +14,5 @@
     </material>
     <material name="green">
-        <color rgba="0 1 0 1" />
+        <color rgba="0 0.5 0 1" />
     </material>
     <material name="black">
@@ -48,5 +48,5 @@
                 <mesh filename="https://raw.githubusercontent.com/Lapland-Robotics/AI.R-Autonomous_Robot/documentation/3D%20Modeling/Snower_whole_3d.stl"/>
             </geometry>
-            <material name="orange" />
+            <material name="green" />
         </visual>
         <collision>
