Commit message: Changed the path type of the snower 3D model file and added a Readme for the explanation of adding the robot package

File: Software/ros2_ws/src/robot/urdf/snower_core.xacro (robot description, xacro)
@@ -46,5 +46,8 @@
             <origin xyz="0 0 -0.245" rpy="0 0 0"/>
             <geometry>
-                <mesh filename="https://raw.githubusercontent.com/Lapland-Robotics/AI.R-Autonomous_Robot/documentation/3D%20Modeling/Snower_whole_3d.stl"/>
+                <!-- Absolute path ▼ -->
+                <!-- <mesh filename="https://raw.githubusercontent.com/Lapland-Robotics/AI.R-Autonomous_Robot/documentation/3D%20Modeling/Snower_whole_3d.stl"/> -->
+                <!-- Relative path ▼ -->
+                <mesh filename="package://robot/urdf/Snower_whole_3d.stl"/>
             </geometry>
             <material name="green" />
